File: PM3_Flash.kicad_pcb (KiCad board)
At the start: 2 copper layers, 10.5 x 11.3 mm, 4 parts, among them J1 Conn_01x02, J2 Conn_01x04, U1 W25Qxx

Commit message: pcb: better layout
Parts:
- moved J1 7.62 mm to (116.2, 65.6), turned to 90 degrees
- moved C1 5.54 mm to (122.8, 65.5)
Routing:
- net GND: track 15.3 -> 13.9 mm, vias 2 -> 5
- net VCC: track 20.3 -> 21.2 mm
- added copper zone on B.Cu, net GND
- added copper zone on F.Cu, net GND
Other:
- board size 10.5 x 11.3 mm -> 10.5 x 11.9 mm
Changed lines of the file:
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@@
   (net 6 "/CLK")
   (footprint "Capacitor_SMD:C_0805_2012Metric_Pad1.18x1.45mm_HandSolder" (layer "F.Cu")
-    (at 117.23 65.5 180)
+    (at 122.77 65.55 180)
     (descr "Capacitor SMD 0805 (2012 Metric), square (rectangular) end terminal, IPC_7351 nominal with elongated pad for handsoldering. (Body size source: IPC-SM-782 page 76, https://www.pcb-3d.com/wordpress/wp-content/uploads/ipc-sm-782a_amendment_1_and_2.pdf, https://docs.google.com/spreadsheets/d/1BsfQQcO9C6DZCsRaXUlFlo91Tg2WpOkGARC1WS5S8t0/edit?usp=sharing), generated with kicad-footprint-generator")
     (tags "capacitor handsolder")
@@
     (fp_text value "10u" (at 0 1.68) (layer "F.Fab")
         (effects (font (size 1 1) (thickness 0.15)))
-    )
-    (fp_text user "${REFERENCE}" (at 0 0) (layer "F.Fab")
-        (effects (font (size 0.5 0.5) (thickness 0.08)))
     )
     (fp_line (start -0.261252 -0.735) (end 0.261252 -0.735)
@@
   )
   (footprint "Connector_PinHeader_2.54mm:PinHeader_1x02_P2.54mm_Vertical" (layer "F.Cu")
-    (at 123.8 65.6 -90)
+    (at 116.18 65.6 90)
     (descr "Through hole straight pin header, 1x02, 2.54mm pitch, single row")
     (tags "Through hole pin header THT 1x02 2.54mm single row")
@@
         (effects (font (size 1 1) (thickness 0.15)))
     )
-    (fp_text user "${REFERENCE}" (at 0 1.27) (layer "F.Fab")
-        (effects (font (size 1 1) (thickness 0.15)))
-    )
     (fp_line (start -1.33 -1.33) (end 0 -1.33)
       (stroke (width 0.12) (type solid)) (layer "F.SilkS"))
@@
     (fp_line (start 1.27 3.81) (end -1.27 3.81)
       (stroke (width 0.1) (type solid)) (layer "F.Fab"))
-    (pad "1" thru_hole rect (at 0 0 270) (size 1.7 1.7) (drill 1) (layers "*.Cu" "*.Mask")
+    (pad "1" thru_hole rect (at 0 0 90) (size 1.7 1.7) (drill 1) (layers "*.Cu" "*.Mask")
       (net 1 "VCC") (pinfunction "Pin_1") (pintype "passive"))
-    (pad "2" thru_hole oval (at 0 2.54 270) (size 1.7 1.7) (drill 1) (layers "*.Cu" "*.Mask")
+    (pad "2" thru_hole oval (at 0 2.54 90) (size 1.7 1.7) (drill 1) (layers "*.Cu" "*.Mask")
       (net 2 "GND") (pinfunction "Pin_2") (pintype "passive"))
     (model "${KICAD6_3DMODEL_DIR}/Connector_PinHeader_2.54mm.3dshapes/PinHeader_1x02_P2.54mm_Vertical.wrl"
@@
   (gr_rect (start 117.62 68.02) (end 117.77 68.17)
     (stroke (width 0.15) (type default)) (fill none) (layer "F.SilkS"))
-  (gr_line (start 115.23 64.33) (end 124.77 64.33)
+  (gr_line (start 115.23 63.73) (end 124.77 63.73)
     (stroke (width 0.1) (type default)) (layer "Edge.Cuts"))
   (gr_line (start 124.77 75.67) (end 115.24 75.67)
@@
   (gr_line (start 125.27 75.17) (end 124.77 75.67)
     (stroke (width 0.1) (type default)) (layer "Edge.Cuts"))
-  (gr_line (start 124.77 64.33) (end 125.27 64.83)
+  (gr_line (start 124.77 63.73) (end 125.27 64.23)
     (stroke (width 0.1) (type default)) (layer "Edge.Cuts"))
   (gr_line (start 114.74 75.17) (end 115.24 75.67)
     (stroke (width 0.1) (type default)) (layer "Edge.Cuts"))
-  (gr_line (start 114.74 75.17) (end 114.73 64.83)
-    (stroke (width 0.1) (type default)) (layer "Edge.Cuts"))
-  (gr_line (start 115.23 64.33) (end 114.73 64.83)
-    (stroke (width 0.1) (type default)) (layer "Edge.Cuts"))
-  (gr_line (start 125.27 64.83) (end 125.27 75.17)
-    (stroke (width 0.1) (type default)) (layer "Edge.Cuts"))
-  (gr_text "VCC" (at 123.8 68.1) (layer "B.SilkS")
+  (gr_line (start 114.74 75.17) (end 114.73 64.23)
+    (stroke (width 0.1) (type default)) (layer "Edge.Cuts"))
+  (gr_line (start 115.23 63.73) (end 114.73 64.23)
+    (stroke (width 0.1) (type default)) (layer "Edge.Cuts"))
+  (gr_line (start 125.27 64.23) (end 125.27 75.17)
+    (stroke (width 0.1) (type default)) (layer "Edge.Cuts"))
+  (gr_text "VCC" (at 116.18 68.1) (layer "B.SilkS")
     (effects (font (size 1 1) (thickness 0.15)) (justify bottom mirror))
   )
@@
     (effects (font (size 1 1) (thickness 0.15)) (justify bottom mirror))
   )
-  (gr_text "G" (at 121.26 68.1) (layer "B.SilkS")
+  (gr_text "G" (at 118.72 68.1) (layer "B.SilkS")
     (effects (font (size 1 1) (thickness 0.15)) (justify bottom mirror))
   )
@@
   (segment (start 117.91 71.3) (end 117.245 70.635) (width 0.4) (layer "F.Cu") (net 1))
   (segment (start 123.6 68.095) (end 123.6 65.8) (width 0.4) (layer "F.Cu") (net 1))
-  (segment (start 120.8625 68.095) (end 118.2675 65.5) (width 0.4) (layer "F.Cu") (net 1))
+  (segment (start 117.5 64.28) (end 122.5375 64.28) (width 0.4) (layer "F.Cu") (net 1))
+  (segment (start 116.18 65.6) (end 117.5 64.28) (width 0.4) (layer "F.Cu") (net 1))
   (segment (start 117.245 70.635) (end 116.4 70.635) (width 0.4) (layer "F.Cu") (net 1))
   (segment (start 123.6 68.095) (end 123.6 69.365) (width 0.4) (layer "F.Cu") (net 1))
-  (segment (start 123.6 65.8) (end 123.8 65.6) (width 0.4) (layer "F.Cu") (net 1))
-  (segment (start 123.6 68.095) (end 120.8625 68.095) (width 0.4) (layer "F.Cu") (net 1))
+  (segment (start 122.5375 64.28) (end 123.8075 65.55) (width 0.4) (layer "F.Cu") (net 1))
   (via (at 117.91 71.3) (size 0.8) (drill 0.4) (layers "F.Cu" "B.Cu") (net 1))
-  (segment (start 117.91 71.3) (end 118.1 71.3) (width 0.4) (layer "B.Cu") (net 1))
-  (segment (start 118.1 71.3) (end 123.8 65.6) (width 0.4) (layer "B.Cu") (net 1))
-  (segment (start 116.37 65.5) (end 118.23 67.36) (width 0.4) (layer "F.Cu") (net 2))
+  (segment (start 116.18 65.6) (end 118.84 68.26) (width 0.4) (layer "B.Cu") (net 1))
+  (segment (start 118.84 68.26) (end 118.84 70.37) (width 0.4) (layer "B.Cu") (net 1))
+  (segment (start 118.84 70.37) (end 117.91 71.3) (width 0.4) (layer "B.Cu") (net 1))
+  (segment (start 118.72 65.6) (end 121.6825 65.6) (width 0.4) (layer "F.Cu") (net 2))
+  (segment (start 116.845 71.905) (end 117.91 72.97) (width 0.4) (layer "F.Cu") (net 2))
+  (segment (start 121.733 67.9) (end 121.733 65.5505) (width 0.4) (layer "F.Cu") (net 2))
   (segment (start 116.4 71.905) (end 116.845 71.905) (width 0.4) (layer "F.Cu") (net 2))
-  (segment (start 116.845 71.905) (end 117.91 72.97) (width 0.4) (layer "F.Cu") (net 2))
-  (segment (start 116.1925 65.5) (end 116.37 65.5) (width 0.4) (layer "F.Cu") (net 2))
+  (segment (start 121.733 65.5505) (end 121.7325 65.55) (width 0.4) (layer "F.Cu") (net 2))
+  (via (at 121.12 71.81) (size 0.8) (drill 0.4) (layers "F.Cu" "B.Cu") (net 2))
   (via (at 117.91 72.97) (size 0.8) (drill 0.4) (layers "F.Cu" "B.Cu") (net 2))
-  (via (at 118.23 67.36) (size 0.8) (drill 0.4) (layers "F.Cu" "B.Cu") (net 2))
-  (segment (start 119.5 67.36) (end 121.26 65.6) (width 0.4) (layer "B.Cu") (net 2))
-  (segment (start 116.66 68.93) (end 116.66 71.72) (width 0.4) (layer "B.Cu") (net 2))
-  (segment (start 116.66 71.72) (end 117.91 72.97) (width 0.4) (layer "B.Cu") (net 2))
-  (segment (start 118.23 67.36) (end 116.66 68.93) (width 0.4) (layer "B.Cu") (net 2))
-  (segment (start 118.23 67.36) (end 119.5 67.36) (width 0.4) (layer "B.Cu") (net 2))
+  (via (at 121.733 67.9) (size 0.8) (drill 0.4) (layers "F.Cu" "B.Cu") (net 2))
+  (via (at 117.89 68.73) (size 0.8) (drill 0.4) (layers "F.Cu" "B.Cu") (net 2))
+  (via (at 121.9 70.4) (size 0.8) (drill 0.4) (layers "F.Cu" "B.Cu") (net 2))
+  (segment (start 121.733 69.147) (end 117.91 72.97) (width 0.4) (layer "B.Cu") (net 2))
+  (segment (start 121.733 69.147) (end 121.733 67.9) (width 0.4) (layer "B.Cu") (net 2))
   (segment (start 115.19 68.84) (end 115.19 73.41) (width 0.3) (layer "F.Cu") (net 3))
   (segment (start 115.935 68.095) (end 115.19 68.84) (width 0.3) (layer "F.Cu") (net 3))
@@
   (segment (start 124.8 71.36) (end 124.8 73.4) (width 0.3) (layer "F.Cu") (net 6))
   (segment (start 124.8 73.4) (end 123.8 74.4) (width 0.3) (layer "F.Cu") (net 6))
+  (zone (net 0) (net_name "") (layer "F.Cu") (hatch edge 0.5)
+    (connect_pads (clearance 0))
+    (min_thickness 0.25) (filled_areas_thickness no)
+    (keepout (tracks allowed) (vias allowed) (pads allowed) (copperpour not_allowed) (footprints allowed))
+    (fill (thermal_gap 0.5) (thermal_bridge_width 0.5))
+    (polygon
+      (pts
+        (xy 117.7 73)
+        (xy 117.7 72.08)
+        (xy 118.2 72.08)
+        (xy 118.2 73)
+      )
+    )
+  )
+  (zone (net 2) (net_name "GND") (layer "F.Cu") (hatch edge 0.5)
+    (connect_pads (clearance 0.4))
+    (min_thickness 0.25) (filled_areas_thickness no)
+    (fill yes (thermal_gap 0.5) (thermal_bridge_width 0.5))
+    (polygon
+      (pts
+        (xy 117.7 67.1)
+        (xy 122.3 67.1)
+        (xy 122.3 73)
+        (xy 117.7 73)
+      )
+    )
+  )
+  (zone (net 2) (net_name "GND") (layer "B.Cu") (hatch edge 0.5)
+    (connect_pads (clearance 0.4))
+    (min_thickness 0.25) (filled_areas_thickness no)
+    (fill yes (thermal_gap 0.5) (thermal_bridge_width 0.5))
+    (polygon
+      (pts
+        (xy 114.73 67.1)
+        (xy 125.27 67.1)
+        (xy 125.27 75.67)
+        (xy 114.73 75.67)
+      )
+    )
+  )
 )

Commit message: 10uF->100nF
Parts:
- C1: value 10u -> 100n
Changed lines of the file:
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@@
         (effects (font (size 1 1) (thickness 0.15)))
     )
-    (fp_text value "10u" (at 0 1.68) (layer "F.Fab")
+    (fp_text value "100n" (at 0 1.68) (layer "F.Fab")
         (effects (font (size 1 1) (thickness 0.15)))
     )
